File: PCB/FaikoutETH/Faikout.kicad_pcb (KiCad board)
At the start: 2 copper layers, 70 x 70 mm, 73 parts, among them J1 1x5, J2 TC2030-USB-NL, J3 Reset, J4 RJ45_LED, Q1 BSS138PS, U1 KSZ8851SNL, U2 TPS62933, U4 ESP32-S3-MINI-1, Y1 Crystal_GND24

Commit message: Revised Ethernet footprint
Routing:
- net GND: track 23.0 -> 31.5 mm

Commit message: More work on Ethernet footprint
Parts:
- moved C10 0.41 mm to (125.8, 78.8), turned to 0 degrees
- moved C20 0.23 mm to (129.2, 65.5), turned to 90 degrees
- moved R7 0.20 mm to (130.4, 65.5)
- moved D6 0.18 mm to (129.8, 65.5)
- moved D5 0.11 mm to (131.0, 65.5)
Routing:
- net +1V8: track 16.4 -> 18.4 mm
- net INTR: track 35.1 -> 36.7 mm
- net VDDIO: track 32.7 -> 33.9 mm
- net GND: track 31.5 -> 32.7 mm, vias 88 -> 91
- net SI: track 29.9 -> 28.9 mm
